Commit message: Update simulation files

File: src/mobileman_simulation/urdf/base_footprint.xacro (robot description, xacro)
@@ -4,6 +4,6 @@
         name = "base_footprint"></link>
     <joint name="base_foot_joint" type="fixed" >
-        <parent link="base_footprint" />
-        <child link="${base_link}" />
+        <child link="base_footprint" />
+        <parent link="${base_link}" />
         <origin xyz="0 0 -0.2155" rpy="0 0 0" />
     </joint>

File: src/mobileman_simulation/urdf/hokuyo_sim.xacro (robot description, xacro)
@@ -32,5 +32,5 @@
       </ray>
       <plugin name="laser" filename="libgazebo_ros_laser.so">
-        <topicName>/laser/scan</topicName>
+        <topicName>/gazebo/scan</topicName>
         <frameName>hokuyo_link</frameName>
       </plugin>

File: src/mobileman_simulation/urdf/imu_sim.xacro (robot description, xacro)
@@ -8,5 +8,5 @@
       <visualize>true</visualize>
       <plugin filename="libgazebo_ros_imu_sensor.so" name="imu_plugin">
-        <topicName>/imu/data</topicName>
+        <topicName>/gazebo/imu/data</topicName>
         <bodyName>imu_link</bodyName>
         <updateRateHZ>100.0</updateRateHZ>
