Commit message: Test - Fix broken packages - "leica_gazebo_simulation" - "leica_scanstation" - "aws-robomaker-hospital-world"

File: src/mobileman_simulation/.history/urdf/mobileman_gazebo_20220510150812.xacro (robot description, xacro)
@@ -103,5 +103,5 @@
     <!--    either differtial_drive_controller should be used or the transmission should be used. -->
     <xacro:include filename="$(find mobileman_simulation)/urdf/differential_drive_controller.xacro" />
-    <transmission name="left_wheel">
+    <!-- <transmission name="left_wheel">
       <type>transmission_interface/SimpleTransmission</type>
       <joint name="front_left_joint">
@@ -120,8 +120,8 @@
         <mechanicalReduction>50</mechanicalReduction>
       </actuator>
-    </transmission>
+    </transmission> -->
     <transmission name="3d_scanner">
       <type>transmission_interface/SimpleTransmission</type>
-      <joint name="photoneo_pan_joint">
+      <joint name="photoneo_tilt_joint">
         <hardwareInterface>hardware_interface/PositionJointInterface</hardwareInterface>
       </joint>
@@ -148,18 +148,18 @@
     <gazebo>
       <plugin name="joint_state_publisher" filename="libgazebo_ros_joint_state_publisher.so">
-        <joint_name>fork_rotational_joint, fork_linear_joint, photoneo_pan_joint, photoneo_tilt_joint, front_left_joint, front_right_joint</joint_name>
+        <joint_name>fork_rotational_joint, fork_linear_joint, photoneo_3d_scanner_joint, front_left_joint, front_right_joint, rear_left_joint, rear_right_joint</joint_name>
       </plugin>
     </gazebo>
     <gazebo reference="front_left_joint">
-      <mu1 value="200.0" />
-      <mu2 value="100.0" />
-      <kp value="5000000.0" />
+      <mu1 value="1.0" />
+      <mu2 value="1.0" />
+      <kp value="1000000.0" />
       <kd value="1.0" />
       <!-- <material>Gazebo/Blue</material> -->
     </gazebo>
     <gazebo reference="front_right_joint">
-      <mu1 value="200.0" />
-      <mu2 value="100.0" />
-      <kp value="5000000.0" />
+      <mu1 value="1.0" />
+      <mu2 value="1.0" />
+      <kp value="1000000.0" />
       <kd value="1.0" />
       <!-- <material>Gazebo/Blue</material> -->

File: src/mobileman_simulation/.history/urdf/mobileman_gazebo_20220510150816.xacro (robot description, xacro)
@@ -103,5 +103,5 @@
     <!--    either differtial_drive_controller should be used or the transmission should be used. -->
     <xacro:include filename="$(find mobileman_simulation)/urdf/differential_drive_controller.xacro" />
-    <transmission name="left_wheel">
+    <!-- <transmission name="left_wheel">
       <type>transmission_interface/SimpleTransmission</type>
       <joint name="front_left_joint">
@@ -120,5 +120,5 @@
         <mechanicalReduction>50</mechanicalReduction>
       </actuator>
-    </transmission>
+    </transmission> -->
     <transmission name="3d_scanner">
       <type>transmission_interface/SimpleTransmission</type>
@@ -148,18 +148,18 @@
     <gazebo>
       <plugin name="joint_state_publisher" filename="libgazebo_ros_joint_state_publisher.so">
-        <joint_name>fork_rotational_joint, fork_linear_joint, photoneo_pan_joint, photoneo_tilt_joint, front_left_joint, front_right_joint</joint_name>
+        <joint_name>fork_rotational_joint, fork_linear_joint, photoneo_3d_scanner_joint, front_left_joint, front_right_joint, rear_left_joint, rear_right_joint</joint_name>
       </plugin>
     </gazebo>
     <gazebo reference="front_left_joint">
-      <mu1 value="200.0" />
-      <mu2 value="100.0" />
-      <kp value="5000000.0" />
+      <mu1 value="1.0" />
+      <mu2 value="1.0" />
+      <kp value="1000000.0" />
       <kd value="1.0" />
       <!-- <material>Gazebo/Blue</material> -->
     </gazebo>
     <gazebo reference="front_right_joint">
-      <mu1 value="200.0" />
-      <mu2 value="100.0" />
-      <kp value="5000000.0" />
+      <mu1 value="1.0" />
+      <mu2 value="1.0" />
+      <kp value="1000000.0" />
       <kd value="1.0" />
       <!-- <material>Gazebo/Blue</material> -->

File: src/mobileman_simulation/.history/urdf/mobileman_gazebo_20220510150843.xacro (robot description, xacro)
@@ -103,5 +103,5 @@
     <!--    either differtial_drive_controller should be used or the transmission should be used. -->
     <xacro:include filename="$(find mobileman_simulation)/urdf/differential_drive_controller.xacro" />
-    <transmission name="left_wheel">
+    <!-- <transmission name="left_wheel">
       <type>transmission_interface/SimpleTransmission</type>
       <joint name="front_left_joint">
@@ -120,5 +120,5 @@
         <mechanicalReduction>50</mechanicalReduction>
       </actuator>
-    </transmission>
+    </transmission> -->
     <transmission name="3d_scanner">
       <type>transmission_interface/SimpleTransmission</type>
@@ -148,18 +148,18 @@
     <gazebo>
       <plugin name="joint_state_publisher" filename="libgazebo_ros_joint_state_publisher.so">
-        <joint_name>fork_rotational_joint, fork_linear_joint, photoneo_pan_joint, photoneo_tilt_joint, front_left_joint, front_right_joint</joint_name>
+        <joint_name>fork_rotational_joint, fork_linear_joint, photoneo_pan_joint, photoneo_tilt_joint, front_left_joint, front_right_joint, rear_left_joint, rear_right_joint</joint_name>
       </plugin>
     </gazebo>
     <gazebo reference="front_left_joint">
-      <mu1 value="200.0" />
-      <mu2 value="100.0" />
-      <kp value="5000000.0" />
+      <mu1 value="1.0" />
+      <mu2 value="1.0" />
+      <kp value="1000000.0" />
       <kd value="1.0" />
       <!-- <material>Gazebo/Blue</material> -->
     </gazebo>
     <gazebo reference="front_right_joint">
-      <mu1 value="200.0" />
-      <mu2 value="100.0" />
-      <kp value="5000000.0" />
+      <mu1 value="1.0" />
+      <mu2 value="1.0" />
+      <kp value="1000000.0" />
       <kd value="1.0" />
       <!-- <material>Gazebo/Blue</material> -->

File: src/mobileman_simulation/.history/urdf/mobileman_gazebo_20220511092449.xacro (robot description, xacro)
@@ -148,18 +148,18 @@
     <gazebo>
       <plugin name="joint_state_publisher" filename="libgazebo_ros_joint_state_publisher.so">
-        <joint_name>fork_rotational_joint, fork_linear_joint, photoneo_pan_joint, photoneo_tilt_joint, front_left_joint, front_right_joint</joint_name>
+        <joint_name>fork_rotational_joint, fork_linear_joint, photoneo_pan_joint, photoneo_tilt_joint, front_left_joint, front_right_joint, rear_left_joint, rear_right_joint</joint_name>
       </plugin>
     </gazebo>
     <gazebo reference="front_left_joint">
-      <mu1 value="200.0" />
-      <mu2 value="100.0" />
-      <kp value="5000000.0" />
+      <mu1 value="1.0" />
+      <mu2 value="1.0" />
+      <kp value="1000000.0" />
       <kd value="1.0" />
       <!-- <material>Gazebo/Blue</material> -->
     </gazebo>
     <gazebo reference="front_right_joint">
-      <mu1 value="200.0" />
-      <mu2 value="100.0" />
-      <kp value="5000000.0" />
+      <mu1 value="1.0" />
+      <mu2 value="1.0" />
+      <kp value="1000000.0" />
       <kd value="1.0" />
       <!-- <material>Gazebo/Blue</material> -->

File: src/mobileman_simulation/.history/urdf/mobileman_gazebo_20220511092836.xacro (robot description, xacro)
@@ -152,14 +152,14 @@
     </gazebo>
     <gazebo reference="front_left_joint">
-      <mu1 value="200.0" />
-      <mu2 value="100.0" />
-      <kp value="5000000.0" />
+      <mu1 value="1.0" />
+      <mu2 value="1.0" />
+      <kp value="1000000.0" />
       <kd value="1.0" />
       <!-- <material>Gazebo/Blue</material> -->
     </gazebo>
     <gazebo reference="front_right_joint">
-      <mu1 value="200.0" />
-      <mu2 value="100.0" />
-      <kp value="5000000.0" />
+      <mu1 value="1.0" />
+      <mu2 value="1.0" />
+      <kp value="1000000.0" />
       <kd value="1.0" />
       <!-- <material>Gazebo/Blue</material> -->

File: src/mobileman_simulation/.history/urdf/mobileman_gazebo_20220511093110.xacro (robot description, xacro)
@@ -151,18 +151,18 @@
       </plugin>
     </gazebo>
-    <gazebo reference="front_left_joint">
-      <mu1 value="200.0" />
-      <mu2 value="100.0" />
-      <kp value="5000000.0" />
+    <!-- <gazebo reference="front_left_joint">
+      <mu1 value="1.0" />
+      <mu2 value="1.0" />
+      <kp value="1000000.0" />
       <kd value="1.0" />
       <!-- <material>Gazebo/Blue</material> -->
     </gazebo>
     <gazebo reference="front_right_joint">
-      <mu1 value="200.0" />
-      <mu2 value="100.0" />
-      <kp value="5000000.0" />
+      <mu1 value="1.0" />
+      <mu2 value="1.0" />
+      <kp value="1000000.0" />
       <kd value="1.0" />
       <!-- <material>Gazebo/Blue</material> -->
-    </gazebo>
+    </gazebo> -->
   </xacro:if>
 </robot>

File: src/mobileman_simulation/.history/urdf/mobileman_gazebo_20220511093150.xacro (robot description, xacro)
@@ -151,18 +151,4 @@
       </plugin>
     </gazebo>
-    <gazebo reference="front_left_joint">
-      <mu1 value="200.0" />
-      <mu2 value="100.0" />
-      <kp value="5000000.0" />
-      <kd value="1.0" />
-      <!-- <material>Gazebo/Blue</material> -->
-    </gazebo>
-    <gazebo reference="front_right_joint">
-      <mu1 value="200.0" />
-      <mu2 value="100.0" />
-      <kp value="5000000.0" />
-      <kd value="1.0" />
-      <!-- <material>Gazebo/Blue</material> -->
-    </gazebo>
   </xacro:if>
 </robot>

File: src/mobileman_simulation/.history/urdf/mobileman_gazebo_20220511093326.xacro (robot description, xacro)
@@ -152,7 +152,7 @@
     </gazebo>
     <gazebo reference="front_left_joint">
-      <mu1 value="200.0" />
-      <mu2 value="100.0" />
-      <kp value="5000000.0" />
+      <mu1 value="1.0" />
+      <mu2 value="1.0" />
+      <kp value="1000000.0" />
       <kd value="1.0" />
       <!-- <material>Gazebo/Blue</material> -->

File: src/mobileman_simulation/.history/urdf/photoneo_3d_scanner_20220510140348.xacro (robot description, xacro)
@@ -1,28 +1,5 @@
 <?xml version="1.0" encoding="UTF-8"?>
 <robot xmlns:xacro="http://www.ros.org/wiki/xacro" name="c5_xacro">
-    <!-- Photoneo Scanner's rotating (pan) mechanism -->
-    <link name="photoneo_pan_link">
-        <inertial>
-            <origin xyz="0 0 0" rpy="0 0 0" />
-            <mass value="3.0" />
-            <inertia ixx="0" ixy="0" ixz="0" iyy="0" iyz="0" izz="6E-04" />
-        </inertial>
-        <visual>
-            <origin xyz="0 0 0" rpy="0 0 0" />
-            <geometry>
-                <cylinder radius="0.02" length="0.51" />
-            </geometry>
-        </visual>
-        <collision>
-            <origin xyz="0 0 0" rpy="0 0 0" />
-            <geometry>
-                <cylinder radius="0.02" length="0.48" />
-            </geometry>
-        </collision>
-    </link>
-    <gazebo reference="photoneo_pan_link">
-        <material>Gazebo/DarkGrey</material>
-    </gazebo>
-    <!--Photoneo (PhoXi) 3D Scanner (M) - body -->
+    <!-- Scanner's rotating (pan) mechanism -->
     <link name="c5_link">
         <inertial>
@@ -44,17 +21,30 @@
         </collision>
     </link>
-    <joint name="photoneo_pan_joint" type="revolute">
-        <origin xyz="0.48 -0.55 -0.16" rpy="0 1.571 0" />
+    <!--PhoXi 3D Scanner (M) - body -->
+    <link name="c5_link">
+        <inertial>
+            <origin xyz="0.011952 0.0002462 -6.0567E-05" rpy="0 0 0" />
+            <mass value="0.8" />
+            <inertia ixx="4.1058E-05" ixy="3.6778E-07" ixz="-1.7672E-09" iyy="5.9376E-06" iyz="-4.2174E-09" izz="4.1185E-05" />
+        </inertial>
+        <visual>
+            <origin xyz="0 0 0" rpy="0 0 0" />
+            <geometry>
+                <box size="0.068 0.416 0.077" />
+            </geometry>
+        </visual>
+        <collision>
+            <origin xyz="0 0 0" rpy="0 0 0" />
+            <geometry>
+                <box size="0.1 0.1 0.02" />
+            </geometry>
+        </collision>
+    </link>
+    <joint name="photoneo_3d_scanner_joint" type="revolute">
+        <origin xyz="0.79 -0.55 -0.19" rpy="0 1.571 0" />
         <parent link="Link2" />
-        <child link="photoneo_pan_link" />
+        <child link="c5_link" />
         <axis xyz="0 0 1" />
-        <limit lower="-0.9" upper="0.9" effort="50" velocity="10" />
-    </joint>
-    <joint name="photoneo_tilt_joint" type="revolute">
-        <origin xyz="0 0 0.33" rpy="0 0 0" />
-        <parent link="photoneo_pan_link" />
-        <child link="c5_link" />
-        <axis xyz="0 1 0" />
-        <limit lower="-0.8" upper="0.6" effort="50" velocity="10" />
+        <limit lower="-0.6" upper="0.9" effort="50" velocity="10" />
     </joint>
     <gazebo reference="c5_link">

File: src/mobileman_simulation/.history/urdf/photoneo_3d_scanner_20220510140534.xacro (robot description, xacro)
@@ -4,12 +4,12 @@
     <link name="photoneo_pan_link">
         <inertial>
-            <origin xyz="0 0 0" rpy="0 0 0" />
-            <mass value="3.0" />
-            <inertia ixx="0" ixy="0" ixz="0" iyy="0" iyz="0" izz="6E-04" />
+            <origin xyz="0.011952 0.0002462 -6.0567E-05" rpy="0 0 0" />
+            <mass value="0.8" />
+            <inertia ixx="4.1058E-05" ixy="3.6778E-07" ixz="-1.7672E-09" iyy="5.9376E-06" iyz="-4.2174E-09" izz="4.1185E-05" />
         </inertial>
         <visual>
             <origin xyz="0 0 0" rpy="0 0 0" />
             <geometry>
-                <cylinder radius="0.02" length="0.51" />
+                <box size="0.068 0.416 0.077" />
             </geometry>
         </visual>
@@ -17,11 +17,8 @@
             <origin xyz="0 0 0" rpy="0 0 0" />
             <geometry>
-                <cylinder radius="0.02" length="0.48" />
+                <<cylinder radius="0.1" length="0.79"/>
             </geometry>
         </collision>
     </link>
-    <gazebo reference="photoneo_pan_link">
-        <material>Gazebo/DarkGrey</material>
-    </gazebo>
     <!--Photoneo (PhoXi) 3D Scanner (M) - body -->
     <link name="c5_link">
@@ -44,17 +41,10 @@
         </collision>
     </link>
-    <joint name="photoneo_pan_joint" type="revolute">
-        <origin xyz="0.48 -0.55 -0.16" rpy="0 1.571 0" />
+    <joint name="photoneo_3d_scanner_joint" type="revolute">
+        <origin xyz="0.79 -0.55 -0.19" rpy="0 1.571 0" />
         <parent link="Link2" />
-        <child link="photoneo_pan_link" />
+        <child link="c5_link" />
         <axis xyz="0 0 1" />
-        <limit lower="-0.9" upper="0.9" effort="50" velocity="10" />
-    </joint>
-    <joint name="photoneo_tilt_joint" type="revolute">
-        <origin xyz="0 0 0.33" rpy="0 0 0" />
-        <parent link="photoneo_pan_link" />
-        <child link="c5_link" />
-        <axis xyz="0 1 0" />
-        <limit lower="-0.8" upper="0.6" effort="50" velocity="10" />
+        <limit lower="-0.6" upper="0.9" effort="50" velocity="10" />
     </joint>
     <gazebo reference="c5_link">

File: src/mobileman_simulation/.history/urdf/photoneo_3d_scanner_20220510140622.xacro (robot description, xacro)
@@ -4,12 +4,12 @@
     <link name="photoneo_pan_link">
         <inertial>
-            <origin xyz="0 0 0" rpy="0 0 0" />
-            <mass value="3.0" />
-            <inertia ixx="0" ixy="0" ixz="0" iyy="0" iyz="0" izz="6E-04" />
+            <origin xyz="0.011952 0.0002462 -6.0567E-05" rpy="0 0 0" />
+            <mass value="1.0" />
+            <inertia ixx="4.1058E-05" ixy="3.6778E-07" ixz="-1.7672E-09" iyy="5.9376E-06" iyz="-4.2174E-09" izz="4.1185E-05" />
         </inertial>
         <visual>
             <origin xyz="0 0 0" rpy="0 0 0" />
             <geometry>
-                <cylinder radius="0.02" length="0.51" />
+                <box size="0.068 0.416 0.077" />
             </geometry>
         </visual>
@@ -17,11 +17,8 @@
             <origin xyz="0 0 0" rpy="0 0 0" />
             <geometry>
-                <cylinder radius="0.02" length="0.48" />
+                <<cylinder radius="0.1" length="0.79"/>
             </geometry>
         </collision>
     </link>
-    <gazebo reference="photoneo_pan_link">
-        <material>Gazebo/DarkGrey</material>
-    </gazebo>
     <!--Photoneo (PhoXi) 3D Scanner (M) - body -->
     <link name="c5_link">
@@ -44,17 +41,10 @@
         </collision>
     </link>
-    <joint name="photoneo_pan_joint" type="revolute">
-        <origin xyz="0.48 -0.55 -0.16" rpy="0 1.571 0" />
+    <joint name="photoneo_3d_scanner_joint" type="revolute">
+        <origin xyz="0.79 -0.55 -0.19" rpy="0 1.571 0" />
         <parent link="Link2" />
-        <child link="photoneo_pan_link" />
+        <child link="c5_link" />
         <axis xyz="0 0 1" />
-        <limit lower="-0.9" upper="0.9" effort="50" velocity="10" />
-    </joint>
-    <joint name="photoneo_tilt_joint" type="revolute">
-        <origin xyz="0 0 0.33" rpy="0 0 0" />
-        <parent link="photoneo_pan_link" />
-        <child link="c5_link" />
-        <axis xyz="0 1 0" />
-        <limit lower="-0.8" upper="0.6" effort="50" velocity="10" />
+        <limit lower="-0.6" upper="0.9" effort="50" velocity="10" />
     </joint>
     <gazebo reference="c5_link">

File: src/mobileman_simulation/.history/urdf/photoneo_3d_scanner_20220510140642.xacro (robot description, xacro)
@@ -5,11 +5,11 @@
         <inertial>
             <origin xyz="0 0 0" rpy="0 0 0" />
-            <mass value="3.0" />
-            <inertia ixx="0" ixy="0" ixz="0" iyy="0" iyz="0" izz="6E-04" />
+            <mass value="1.0" />
+            <inertia ixx="4.1058E-05" ixy="3.6778E-07" ixz="-1.7672E-09" iyy="5.9376E-06" iyz="-4.2174E-09" izz="4.1185E-05" />
         </inertial>
         <visual>
             <origin xyz="0 0 0" rpy="0 0 0" />
             <geometry>
-                <cylinder radius="0.02" length="0.51" />
+                <box size="0.068 0.416 0.077" />
             </geometry>
         </visual>
@@ -17,11 +17,8 @@
             <origin xyz="0 0 0" rpy="0 0 0" />
             <geometry>
-                <cylinder radius="0.02" length="0.48" />
+                <<cylinder radius="0.1" length="0.79"/>
             </geometry>
         </collision>
     </link>
-    <gazebo reference="photoneo_pan_link">
-        <material>Gazebo/DarkGrey</material>
-    </gazebo>
     <!--Photoneo (PhoXi) 3D Scanner (M) - body -->
     <link name="c5_link">
@@ -44,17 +41,10 @@
         </collision>
     </link>
-    <joint name="photoneo_pan_joint" type="revolute">
-        <origin xyz="0.48 -0.55 -0.16" rpy="0 1.571 0" />
+    <joint name="photoneo_3d_scanner_joint" type="revolute">
+        <origin xyz="0.79 -0.55 -0.19" rpy="0 1.571 0" />
         <parent link="Link2" />
-        <child link="photoneo_pan_link" />
+        <child link="c5_link" />
         <axis xyz="0 0 1" />
-        <limit lower="-0.9" upper="0.9" effort="50" velocity="10" />
-    </joint>
-    <joint name="photoneo_tilt_joint" type="revolute">
-        <origin xyz="0 0 0.33" rpy="0 0 0" />
-        <parent link="photoneo_pan_link" />
-        <child link="c5_link" />
-        <axis xyz="0 1 0" />
-        <limit lower="-0.8" upper="0.6" effort="50" velocity="10" />
+        <limit lower="-0.6" upper="0.9" effort="50" velocity="10" />
     </joint>
     <gazebo reference="c5_link">

File: src/mobileman_simulation/.history/urdf/photoneo_3d_scanner_20220510140705.xacro (robot description, xacro)
@@ -5,11 +5,11 @@
         <inertial>
             <origin xyz="0 0 0" rpy="0 0 0" />
-            <mass value="3.0" />
-            <inertia ixx="0" ixy="0" ixz="0" iyy="0" iyz="0" izz="6E-04" />
+            <mass value="1.0" />
+            <inertia ixx="4.1058E-05" ixy="3.6778E-07" ixz="-1.7672E-09" iyy="5.9376E-06" iyz="-4.2174E-09" izz="4.1185E-05" />
         </inertial>
         <visual>
             <origin xyz="0 0 0" rpy="0 0 0" />
             <geometry>
-                <cylinder radius="0.02" length="0.51" />
+                <<cylinder radius="0.1" length="0.79"/>
             </geometry>
         </visual>
@@ -17,11 +17,8 @@
             <origin xyz="0 0 0" rpy="0 0 0" />
             <geometry>
-                <cylinder radius="0.02" length="0.48" />
+                <<cylinder radius="0.1" length="0.79"/>
             </geometry>
         </collision>
     </link>
-    <gazebo reference="photoneo_pan_link">
-        <material>Gazebo/DarkGrey</material>
-    </gazebo>
     <!--Photoneo (PhoXi) 3D Scanner (M) - body -->
     <link name="c5_link">
@@ -44,17 +41,10 @@
         </collision>
     </link>
-    <joint name="photoneo_pan_joint" type="revolute">
-        <origin xyz="0.48 -0.55 -0.16" rpy="0 1.571 0" />
+    <joint name="photoneo_3d_scanner_joint" type="revolute">
+        <origin xyz="0.79 -0.55 -0.19" rpy="0 1.571 0" />
         <parent link="Link2" />
-        <child link="photoneo_pan_link" />
+        <child link="c5_link" />
         <axis xyz="0 0 1" />
-        <limit lower="-0.9" upper="0.9" effort="50" velocity="10" />
-    </joint>
-    <joint name="photoneo_tilt_joint" type="revolute">
-        <origin xyz="0 0 0.33" rpy="0 0 0" />
-        <parent link="photoneo_pan_link" />
-        <child link="c5_link" />
-        <axis xyz="0 1 0" />
-        <limit lower="-0.8" upper="0.6" effort="50" velocity="10" />
+        <limit lower="-0.6" upper="0.9" effort="50" velocity="10" />
     </joint>
     <gazebo reference="c5_link">
