Commit message: Test - Fix broken packages - "leica_gazebo_simulation" - "leica_scanstation" - "aws-robomaker-hospital-world"

File: src/mobileman_simulation/.history/urdf/photoneo_3d_scanner_20220510141133.xacro (robot description, xacro)
@@ -5,11 +5,11 @@
         <inertial>
             <origin xyz="0 0 0" rpy="0 0 0" />
-            <mass value="3.0" />
-            <inertia ixx="0" ixy="0" ixz="0" iyy="0" iyz="0" izz="6E-04" />
+            <mass value="1.0" />
+            <inertia ixx="4.1058E-05" ixy="3.6778E-07" ixz="-1.7672E-09" iyy="5.9376E-06" iyz="-4.2174E-09" izz="4.1185E-05" />
         </inertial>
         <visual>
             <origin xyz="0 0 0" rpy="0 0 0" />
             <geometry>
-                <cylinder radius="0.02" length="0.51" />
+                <<cylinder radius="0.1" length="0.79"/>
             </geometry>
         </visual>
@@ -17,11 +17,8 @@
             <origin xyz="0 0 0" rpy="0 0 0" />
             <geometry>
-                <cylinder radius="0.02" length="0.48" />
+                <<cylinder radius="0.1" length="0.79"/>
             </geometry>
         </collision>
     </link>
-    <gazebo reference="photoneo_pan_link">
-        <material>Gazebo/DarkGrey</material>
-    </gazebo>
     <!--Photoneo (PhoXi) 3D Scanner (M) - body -->
     <link name="c5_link">
@@ -44,17 +41,17 @@
         </collision>
     </link>
-    <joint name="photoneo_pan_joint" type="revolute">
-        <origin xyz="0.48 -0.55 -0.16" rpy="0 1.571 0" />
+    <joint name="Link2_joint" type="fixed">
+        <origin xyz="0.79 -0.55 -0.19" rpy="0 1.571 0" />
         <parent link="Link2" />
         <child link="photoneo_pan_link" />
         <axis xyz="0 0 1" />
-        <limit lower="-0.9" upper="0.9" effort="50" velocity="10" />
+        <limit lower="-0.6" upper="0.9" effort="50" velocity="10" />
     </joint>
-    <joint name="photoneo_tilt_joint" type="revolute">
-        <origin xyz="0 0 0.33" rpy="0 0 0" />
-        <parent link="photoneo_pan_link" />
+    <joint name="photoneo_3d_scanner_joint" type="revolute">
+        <origin xyz="0.79 -0.55 -0.19" rpy="0 1.571 0" />
+        <parent link="Link2" />
         <child link="c5_link" />
-        <axis xyz="0 1 0" />
-        <limit lower="-0.8" upper="0.6" effort="50" velocity="10" />
+        <axis xyz="0 0 1" />
+        <limit lower="-0.6" upper="0.9" effort="50" velocity="10" />
     </joint>
     <gazebo reference="c5_link">

File: src/mobileman_simulation/.history/urdf/photoneo_3d_scanner_20220510141206.xacro (robot description, xacro)
@@ -5,11 +5,11 @@
         <inertial>
             <origin xyz="0 0 0" rpy="0 0 0" />
-            <mass value="3.0" />
-            <inertia ixx="0" ixy="0" ixz="0" iyy="0" iyz="0" izz="6E-04" />
+            <mass value="1.0" />
+            <inertia ixx="4.1058E-05" ixy="3.6778E-07" ixz="-1.7672E-09" iyy="5.9376E-06" iyz="-4.2174E-09" izz="4.1185E-05" />
         </inertial>
         <visual>
             <origin xyz="0 0 0" rpy="0 0 0" />
             <geometry>
-                <cylinder radius="0.02" length="0.51" />
+                <<cylinder radius="0.1" length="0.79"/>
             </geometry>
         </visual>
@@ -17,11 +17,8 @@
             <origin xyz="0 0 0" rpy="0 0 0" />
             <geometry>
-                <cylinder radius="0.02" length="0.48" />
+                <<cylinder radius="0.1" length="0.79"/>
             </geometry>
         </collision>
     </link>
-    <gazebo reference="photoneo_pan_link">
-        <material>Gazebo/DarkGrey</material>
-    </gazebo>
     <!--Photoneo (PhoXi) 3D Scanner (M) - body -->
     <link name="c5_link">
@@ -44,17 +41,15 @@
         </collision>
     </link>
-    <joint name="photoneo_pan_joint" type="revolute">
-        <origin xyz="0.48 -0.55 -0.16" rpy="0 1.571 0" />
+    <joint name="Link2_joint" type="fixed">
+        <origin xyz="0.79 -0.55 -0.19" rpy="0 1.571 0" />
         <parent link="Link2" />
         <child link="photoneo_pan_link" />
+    </joint>
+    <joint name="photoneo_3d_scanner_joint" type="revolute">
+        <origin xyz="0.79 -0.55 -0.19" rpy="0 1.571 0" />
+        <parent link="Link2" />
+        <child link="c5_link" />
         <axis xyz="0 0 1" />
-        <limit lower="-0.9" upper="0.9" effort="50" velocity="10" />
-    </joint>
-    <joint name="photoneo_tilt_joint" type="revolute">
-        <origin xyz="0 0 0.33" rpy="0 0 0" />
-        <parent link="photoneo_pan_link" />
-        <child link="c5_link" />
-        <axis xyz="0 1 0" />
-        <limit lower="-0.8" upper="0.6" effort="50" velocity="10" />
+        <limit lower="-0.6" upper="0.9" effort="50" velocity="10" />
     </joint>
     <gazebo reference="c5_link">

File: src/mobileman_simulation/.history/urdf/photoneo_3d_scanner_20220510141244.xacro (robot description, xacro)
@@ -5,11 +5,11 @@
         <inertial>
             <origin xyz="0 0 0" rpy="0 0 0" />
-            <mass value="3.0" />
-            <inertia ixx="0" ixy="0" ixz="0" iyy="0" iyz="0" izz="6E-04" />
+            <mass value="1.0" />
+            <inertia ixx="4.1058E-05" ixy="3.6778E-07" ixz="-1.7672E-09" iyy="5.9376E-06" iyz="-4.2174E-09" izz="4.1185E-05" />
         </inertial>
         <visual>
             <origin xyz="0 0 0" rpy="0 0 0" />
             <geometry>
-                <cylinder radius="0.02" length="0.51" />
+                <cylinder radius="0.1" length="0.79"/>
             </geometry>
         </visual>
@@ -17,11 +17,8 @@
             <origin xyz="0 0 0" rpy="0 0 0" />
             <geometry>
-                <cylinder radius="0.02" length="0.48" />
+                <cylinder radius="0.1" length="0.79"/>
             </geometry>
         </collision>
     </link>
-    <gazebo reference="photoneo_pan_link">
-        <material>Gazebo/DarkGrey</material>
-    </gazebo>
     <!--Photoneo (PhoXi) 3D Scanner (M) - body -->
     <link name="c5_link">
@@ -44,17 +41,15 @@
         </collision>
     </link>
-    <joint name="photoneo_pan_joint" type="revolute">
-        <origin xyz="0.48 -0.55 -0.16" rpy="0 1.571 0" />
+    <joint name="Link2_joint" type="fixed">
+        <origin xyz="0.79 -0.55 -0.19" rpy="0 1.571 0" />
         <parent link="Link2" />
         <child link="photoneo_pan_link" />
+    </joint>
+    <joint name="photoneo_3d_scanner_joint" type="revolute">
+        <origin xyz="0.79 -0.55 -0.19" rpy="0 1.571 0" />
+        <parent link="Link2" />
+        <child link="c5_link" />
         <axis xyz="0 0 1" />
-        <limit lower="-0.9" upper="0.9" effort="50" velocity="10" />
-    </joint>
-    <joint name="photoneo_tilt_joint" type="revolute">
-        <origin xyz="0 0 0.33" rpy="0 0 0" />
-        <parent link="photoneo_pan_link" />
-        <child link="c5_link" />
-        <axis xyz="0 1 0" />
-        <limit lower="-0.8" upper="0.6" effort="50" velocity="10" />
+        <limit lower="-0.6" upper="0.9" effort="50" velocity="10" />
     </joint>
     <gazebo reference="c5_link">

File: src/mobileman_simulation/.history/urdf/photoneo_3d_scanner_20220510141357.xacro (robot description, xacro)
@@ -5,11 +5,11 @@
         <inertial>
             <origin xyz="0 0 0" rpy="0 0 0" />
-            <mass value="3.0" />
-            <inertia ixx="0" ixy="0" ixz="0" iyy="0" iyz="0" izz="6E-04" />
+            <mass value="1.0" />
+            <inertia ixx="4.1058E-05" ixy="3.6778E-07" ixz="-1.7672E-09" iyy="5.9376E-06" iyz="-4.2174E-09" izz="4.1185E-05" />
         </inertial>
         <visual>
             <origin xyz="0 0 0" rpy="0 0 0" />
             <geometry>
-                <cylinder radius="0.02" length="0.51" />
+                <cylinder radius="0.1" length="0.79"/>
             </geometry>
         </visual>
@@ -17,11 +17,8 @@
             <origin xyz="0 0 0" rpy="0 0 0" />
             <geometry>
-                <cylinder radius="0.02" length="0.48" />
+                <cylinder radius="0.03" length="0.79"/>
             </geometry>
         </collision>
     </link>
-    <gazebo reference="photoneo_pan_link">
-        <material>Gazebo/DarkGrey</material>
-    </gazebo>
     <!--Photoneo (PhoXi) 3D Scanner (M) - body -->
     <link name="c5_link">
@@ -44,17 +41,15 @@
         </collision>
     </link>
-    <joint name="photoneo_pan_joint" type="revolute">
-        <origin xyz="0.48 -0.55 -0.16" rpy="0 1.571 0" />
+    <joint name="Link2_joint" type="fixed">
+        <origin xyz="0.79 -0.55 -0.19" rpy="0 1.571 0" />
         <parent link="Link2" />
         <child link="photoneo_pan_link" />
+    </joint>
+    <joint name="photoneo_3d_scanner_joint" type="revolute">
+        <origin xyz="0.79 -0.55 -0.19" rpy="0 1.571 0" />
+        <parent link="Link2" />
+        <child link="c5_link" />
         <axis xyz="0 0 1" />
-        <limit lower="-0.9" upper="0.9" effort="50" velocity="10" />
-    </joint>
-    <joint name="photoneo_tilt_joint" type="revolute">
-        <origin xyz="0 0 0.33" rpy="0 0 0" />
-        <parent link="photoneo_pan_link" />
-        <child link="c5_link" />
-        <axis xyz="0 1 0" />
-        <limit lower="-0.8" upper="0.6" effort="50" velocity="10" />
+        <limit lower="-0.6" upper="0.9" effort="50" velocity="10" />
     </joint>
     <gazebo reference="c5_link">

File: src/mobileman_simulation/.history/urdf/photoneo_3d_scanner_20220510141413.xacro (robot description, xacro)
@@ -5,11 +5,11 @@
         <inertial>
             <origin xyz="0 0 0" rpy="0 0 0" />
-            <mass value="3.0" />
-            <inertia ixx="0" ixy="0" ixz="0" iyy="0" iyz="0" izz="6E-04" />
+            <mass value="1.0" />
+            <inertia ixx="4.1058E-05" ixy="3.6778E-07" ixz="-1.7672E-09" iyy="5.9376E-06" iyz="-4.2174E-09" izz="4.1185E-05" />
         </inertial>
         <visual>
             <origin xyz="0 0 0" rpy="0 0 0" />
             <geometry>
-                <cylinder radius="0.02" length="0.51" />
+                <cylinder radius="0.02" length="0.79"/>
             </geometry>
         </visual>
@@ -17,11 +17,8 @@
             <origin xyz="0 0 0" rpy="0 0 0" />
             <geometry>
-                <cylinder radius="0.02" length="0.48" />
+                <cylinder radius="0.02" length="0.79"/>
             </geometry>
         </collision>
     </link>
-    <gazebo reference="photoneo_pan_link">
-        <material>Gazebo/DarkGrey</material>
-    </gazebo>
     <!--Photoneo (PhoXi) 3D Scanner (M) - body -->
     <link name="c5_link">
@@ -44,17 +41,15 @@
         </collision>
     </link>
-    <joint name="photoneo_pan_joint" type="revolute">
-        <origin xyz="0.48 -0.55 -0.16" rpy="0 1.571 0" />
+    <joint name="Link2_joint" type="fixed">
+        <origin xyz="0.79 -0.55 -0.19" rpy="0 1.571 0" />
         <parent link="Link2" />
         <child link="photoneo_pan_link" />
+    </joint>
+    <joint name="photoneo_3d_scanner_joint" type="revolute">
+        <origin xyz="0.79 -0.55 -0.19" rpy="0 1.571 0" />
+        <parent link="Link2" />
+        <child link="c5_link" />
         <axis xyz="0 0 1" />
-        <limit lower="-0.9" upper="0.9" effort="50" velocity="10" />
-    </joint>
-    <joint name="photoneo_tilt_joint" type="revolute">
-        <origin xyz="0 0 0.33" rpy="0 0 0" />
-        <parent link="photoneo_pan_link" />
-        <child link="c5_link" />
-        <axis xyz="0 1 0" />
-        <limit lower="-0.8" upper="0.6" effort="50" velocity="10" />
+        <limit lower="-0.6" upper="0.9" effort="50" velocity="10" />
     </joint>
     <gazebo reference="c5_link">

File: src/mobileman_simulation/.history/urdf/photoneo_3d_scanner_20220510142717.xacro (robot description, xacro)
@@ -2,14 +2,14 @@
 <robot xmlns:xacro="http://www.ros.org/wiki/xacro" name="c5_xacro">
     <!-- Photoneo Scanner's rotating (pan) mechanism -->
-    <link name="photoneo_pan_link">
+    <!-- <link name="photoneo_pan_link">
         <inertial>
             <origin xyz="0 0 0" rpy="0 0 0" />
-            <mass value="3.0" />
-            <inertia ixx="0" ixy="0" ixz="0" iyy="0" iyz="0" izz="6E-04" />
+            <mass value="1.0" />
+            <inertia ixx="4.1058E-05" ixy="3.6778E-07" ixz="-1.7672E-09" iyy="5.9376E-06" iyz="-4.2174E-09" izz="4.1185E-05" />
         </inertial>
         <visual>
             <origin xyz="0 0 0" rpy="0 0 0" />
             <geometry>
-                <cylinder radius="0.02" length="0.51" />
+                <cylinder radius="0.02" length="0.79"/>
             </geometry>
         </visual>
@@ -17,11 +17,8 @@
             <origin xyz="0 0 0" rpy="0 0 0" />
             <geometry>
-                <cylinder radius="0.02" length="0.48" />
+                <cylinder radius="0.02" length="0.79"/>
             </geometry>
         </collision>
-    </link>
-    <gazebo reference="photoneo_pan_link">
-        <material>Gazebo/DarkGrey</material>
-    </gazebo>
+    </link> -->
     <!--Photoneo (PhoXi) 3D Scanner (M) - body -->
     <link name="c5_link">
@@ -44,17 +41,15 @@
         </collision>
     </link>
-    <joint name="photoneo_pan_joint" type="revolute">
-        <origin xyz="0.48 -0.55 -0.16" rpy="0 1.571 0" />
+    <!-- <joint name="Link2_joint" type="fixed">
+        <origin xyz="0.79 -0.55 -0.19" rpy="0 1.571 0" />
         <parent link="Link2" />
         <child link="photoneo_pan_link" />
+    </joint> -->
+    <joint name="photoneo_3d_scanner_joint" type="revolute">
+        <origin xyz="0.79 -0.55 -0.19" rpy="0 1.571 0" />
+        <parent link="Link2" />
+        <child link="c5_link" />
         <axis xyz="0 0 1" />
-        <limit lower="-0.9" upper="0.9" effort="50" velocity="10" />
-    </joint>
-    <joint name="photoneo_tilt_joint" type="revolute">
-        <origin xyz="0 0 0.33" rpy="0 0 0" />
-        <parent link="photoneo_pan_link" />
-        <child link="c5_link" />
-        <axis xyz="0 1 0" />
-        <limit lower="-0.8" upper="0.6" effort="50" velocity="10" />
+        <limit lower="-0.6" upper="0.9" effort="50" velocity="10" />
     </joint>
     <gazebo reference="c5_link">

File: src/mobileman_simulation/.history/urdf/photoneo_3d_scanner_20220510143558.xacro (robot description, xacro)
@@ -5,11 +5,11 @@
         <inertial>
             <origin xyz="0 0 0" rpy="0 0 0" />
-            <mass value="3.0" />
-            <inertia ixx="0" ixy="0" ixz="0" iyy="0" iyz="0" izz="6E-04" />
+            <mass value="1.0" />
+            <inertia ixx="4.1058E-05" ixy="3.6778E-07" ixz="-1.7672E-09" iyy="5.9376E-06" iyz="-4.2174E-09" izz="4.1185E-05" />
         </inertial>
         <visual>
             <origin xyz="0 0 0" rpy="0 0 0" />
             <geometry>
-                <cylinder radius="0.02" length="0.51" />
+                <cylinder radius="0.02" length="0.69"/>
             </geometry>
         </visual>
@@ -17,11 +17,8 @@
             <origin xyz="0 0 0" rpy="0 0 0" />
             <geometry>
-                <cylinder radius="0.02" length="0.48" />
+                <cylinder radius="0.02" length="0.79"/>
             </geometry>
         </collision>
     </link>
-    <gazebo reference="photoneo_pan_link">
-        <material>Gazebo/DarkGrey</material>
-    </gazebo>
     <!--Photoneo (PhoXi) 3D Scanner (M) - body -->
     <link name="c5_link">
@@ -44,17 +41,15 @@
         </collision>
     </link>
-    <joint name="photoneo_pan_joint" type="revolute">
-        <origin xyz="0.48 -0.55 -0.16" rpy="0 1.571 0" />
+    <joint name="Link2_joint" type="fixed">
+        <origin xyz="0.79 -0.55 -0.19" rpy="0 1.571 0" />
         <parent link="Link2" />
         <child link="photoneo_pan_link" />
+    </joint>
+    <joint name="photoneo_3d_scanner_joint" type="revolute">
+        <origin xyz="0.79 -0.55 -0.19" rpy="0 1.571 0" />
+        <parent link="Link2" />
+        <child link="c5_link" />
         <axis xyz="0 0 1" />
-        <limit lower="-0.9" upper="0.9" effort="50" velocity="10" />
-    </joint>
-    <joint name="photoneo_tilt_joint" type="revolute">
-        <origin xyz="0 0 0.33" rpy="0 0 0" />
-        <parent link="photoneo_pan_link" />
-        <child link="c5_link" />
-        <axis xyz="0 1 0" />
-        <limit lower="-0.8" upper="0.6" effort="50" velocity="10" />
+        <limit lower="-0.6" upper="0.9" effort="50" velocity="10" />
     </joint>
     <gazebo reference="c5_link">
